File: AudioAmp.sch (EAGLE design)
At the start: 99 parts, among them X1 22-23-2021, X2 22-23-2021

Commit message: todo: check analog supply grounding
Connections:
- net AMPFAULT: now also P1.16
- net TH-WAR: now also P1.18
Changed lines of the file:
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@@
 <label x="109.22" y="58.42" size="1.778" layer="95"/>
+</segment>
+<segment>
+<pinref part="P1" gate="G$1" pin="18"/>
+<wire x1="35.56" y1="287.02" x2="45.72" y2="287.02" width="0.1524" layer="91"/>
+<label x="40.64" y="287.02" size="1.778" layer="95"/>
 </segment>
 </net>
@@
 <label x="109.22" y="60.96" size="1.778" layer="95"/>
 </segment>
+<segment>
+<pinref part="P1" gate="G$1" pin="16"/>
+<wire x1="35.56" y1="289.56" x2="45.72" y2="289.56" width="0.1524" layer="91"/>
+<label x="40.64" y="289.56" size="1.778" layer="95"/>
+</segment>
 </net>

Commit message: almost done
Parts:
- added SL1: (no value), con-amp-quick:M02
Connections:
- net AGND: now also SL1.1
- net AVDD: now also SL1.2; no longer VOLTAGE.2
Changed lines of the file:
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@@
 <part name="R25" library="rcl" deviceset="R-EU_" device="R1206" value="10k"/>
 <part name="R26" library="rcl" deviceset="R-EU_" device="R1206" value="10k"/>
+<part name="SL1" library="con-amp-quick" deviceset="M02" device=""/>
 </parts>
 <sheets>
@@
 <attribute name="VALUE" x="60.198" y="288.29" size="1.778" layer="96" rot="R270"/>
 </instance>
+<instance part="SL1" gate="G$1" x="25.4" y="127"/>
 </instances>
 <busses>
@@
 <label x="35.56" y="167.64" size="1.778" layer="95"/>
 </segment>
+<segment>
+<pinref part="SL1" gate="G$1" pin="1"/>
+<wire x1="33.02" y1="127" x2="43.18" y2="127" width="0.1524" layer="91"/>
+<label x="40.64" y="127" size="1.778" layer="95"/>
+</segment>
 </net>
 <net name="AVDD" class="0">
@@
 </segment>
 <segment>
-<pinref part="VOLTAGE" gate="1" pin="2"/>
-<wire x1="33.02" y1="142.24" x2="43.18" y2="142.24" width="0.1524" layer="91"/>
-<label x="40.64" y="142.24" size="1.778" layer="95"/>
-</segment>
-</net>
+<pinref part="SL1" gate="G$1" pin="2"/>
+<wire x1="33.02" y1="129.54" x2="43.18" y2="129.54" width="0.1524" layer="91"/>
+<label x="40.64" y="129.54" size="1.778" layer="95"/>
+</segment>
+</net>
