File: AudioAmp.sch (EAGLE design)
At the start: 100 parts, among them X1 22-23-2021, X2 22-23-2021

Commit message: done
Connections:
- new net GND1: VOLTAGE.3
- net VCC3.3: now also VOLTAGE.2; no longer VOLTAGE.3
Changed lines of the file:
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@@
 <attribute name="VALUE" x="80.518" y="171.45" size="1.778" layer="96" rot="R270"/>
 </instance>
-<instance part="GND22" gate="1" x="50.8" y="144.78"/>
+<instance part="GND22" gate="1" x="55.88" y="147.32" rot="R90"/>
 <instance part="GND24" gate="1" x="73.66" y="218.44" rot="R270"/>
 <instance part="R25" gate="G$1" x="58.42" y="284.48" smashed="yes" rot="R270">
@@
 <segment>
 <pinref part="VOLTAGE" gate="1" pin="4"/>
-<wire x1="33.02" y1="147.32" x2="50.8" y2="147.32" width="0.1524" layer="91"/>
+<wire x1="33.02" y1="147.32" x2="53.34" y2="147.32" width="0.1524" layer="91"/>
 <pinref part="GND22" gate="1" pin="GND"/>
 </segment>
@@
 </segment>
 <segment>
-<pinref part="VOLTAGE" gate="1" pin="3"/>
-<wire x1="33.02" y1="144.78" x2="43.18" y2="144.78" width="0.1524" layer="91"/>
-<label x="40.64" y="144.78" size="1.778" layer="95"/>
-</segment>
-<segment>
 <pinref part="R21" gate="G$1" pin="2"/>
 <pinref part="R22" gate="G$1" pin="2"/>
@@
 <wire x1="58.42" y1="292.1" x2="58.42" y2="289.56" width="0.1524" layer="91"/>
 <label x="63.5" y="292.1" size="1.778" layer="95"/>
+</segment>
+<segment>
+<pinref part="VOLTAGE" gate="1" pin="2"/>
+<wire x1="33.02" y1="142.24" x2="43.18" y2="142.24" width="0.1524" layer="91"/>
+<label x="40.64" y="142.24" size="1.778" layer="95"/>
 </segment>
 </net>
@@
 </segment>
 </net>
+<net name="GND1" class="0">
+<segment>
+<pinref part="VOLTAGE" gate="1" pin="3"/>
+<wire x1="33.02" y1="144.78" x2="43.18" y2="144.78" width="0.1524" layer="91"/>
+<label x="40.64" y="144.78" size="1.778" layer="95"/>
+</segment>
+</net>
