File: AudioAmp.brd (EAGLE design)
At the start: 100 x 80 mm, 100 parts, among them X1 22-23-2021, X2 22-23-2021

Commit message: done
Parts:
- moved DIGOUT 1.27 mm to (16.5, 25.4)
- moved R15 0.50 mm to (34.2, 24.8)
- moved AUXANALOG 0.39 mm to (49.5, 2.54)
- moved SL1 0.15 mm to (36.8, 2.54), turned to 180 degrees
- turned C2 to 270 degrees
Connections:
- new net GND1: VOLTAGE.3
- net VCC3.3: now also VOLTAGE.2; no longer VOLTAGE.3
Routing:
- net GND: track 413.7 -> 955.8 mm, vias 9 -> 13
- net VCCSIG: track 35.6 -> 25.0 mm
- net AIN3: track 49.7 -> 43.0 mm
- net N$7: track 8.75 -> 14.5 mm
- net AGND: track 132.2 -> 135.7 mm, vias 0 -> 1
- net VCC3.3: track 237.3 -> 235.0 mm, vias 6 -> 7
- net HPRIGHT: track 37.5 -> 36.6 mm
- net N$6: track 18.6 -> 18.0 mm
- net HPGND: track 37.5 -> 38.0 mm
- added copper zone on layer 1, net GND
- added copper zone on layer 1, net GND1
- added copper zone on layer 16, net GND1
